Commit message: base_footprint & lidar added

File: urdf/hamals_robot.urdf.xacro (robot description, xacro)
@@ -7,4 +7,13 @@
   <xacro:property name="chassis_width"  value="0.156"/>
   <xacro:property name="chassis_height" value="0.09"/>
+  <!-- ===================== -->
+  <!-- BASE FOOTPRINT (Z = 0, zemin referansı) -->
+  <!-- ===================== -->
+  <link name="base_footprint"/>
+  <joint name="base_footprint_joint" type="fixed">
+    <parent link="base_footprint"/>
+    <child link="base_link"/>
+    <origin xyz="0 0 0.045"/>
+  </joint>
   <!-- ===================== -->
   <!-- BASE LINK -->
@@ -26,8 +35,7 @@
     <inertial>
       <mass value="5.0"/>
-      <inertia
-        ixx="0.02" ixy="0" ixz="0"
-        iyy="0.02" iyz="0"
-        izz="0.02"/>
+      <inertia ixx="0.02" ixy="0" ixz="0"
+               iyy="0.02" iyz="0"
+               izz="0.02"/>
     </inertial>
   </link>
@@ -36,46 +44,4 @@
   <!-- ===================== -->
   <link name="left_wheel_link">
-    <!-- 🔴 LASTİK -->
-    <visual>
-      <origin xyz="0 0 0" rpy="1.5708 0 0"/>
-      <geometry>
-        <!-- biraz daha kısa -->
-        <cylinder radius="0.035" length="0.030"/>
-      </geometry>
-      <material name="red_tire">
-        <color rgba="0.85 0.0 0.0 1.0"/>
-      </material>
-    </visual>
-    <!-- ⚪ JANT -->
-    <visual>
-      <!-- çok az dışarı taşır -->
-      <origin xyz="0 0 0.002" rpy="1.5708 0 0"/>
-      <geometry>
-        <cylinder radius="0.020" length="0.040"/>
-      </geometry>
-      <material name="white_rim">
-        <color rgba="1.0 1.0 1.0 1.0"/>
-      </material>
-    </visual>
-    <!-- collision sadece lastik -->
-    <collision>
-      <origin xyz="0 0 0" rpy="1.5708 0 0"/>
-      <geometry>
-        <cylinder radius="0.035" length="0.039"/>
-      </geometry>
-    </collision>
-  </link>
-  <!-- LEFT WHEEL JOINT -->
-  <joint name="left_wheel_joint" type="continuous">
-    <parent link="base_link"/>
-    <child link="left_wheel_link"/>
-    <origin xyz="0 0.095 -0.028"/>
-    <axis xyz="1 0 0"/>
-  </joint>
-  <!-- ===================== -->
-  <!-- RIGHT WHEEL -->
-  <!-- ===================== -->
-  <link name="right_wheel_link">
-    <!-- 🔴 LASTİK -->
     <visual>
       <origin xyz="0 0 0" rpy="1.5708 0 0"/>
@@ -87,5 +53,4 @@
       </material>
     </visual>
-    <!-- ⚪ JANT -->
     <visual>
       <origin xyz="0 0 0.002" rpy="1.5708 0 0"/>
@@ -104,5 +69,39 @@
     </collision>
   </link>
-  <!-- RIGHT WHEEL JOINT -->
+  <joint name="left_wheel_joint" type="continuous">
+    <parent link="base_link"/>
+    <child link="left_wheel_link"/>
+    <origin xyz="0 0.095 -0.028"/>
+    <axis xyz="1 0 0"/>
+  </joint>
+  <!-- ===================== -->
+  <!-- RIGHT WHEEL -->
+  <!-- ===================== -->
+  <link name="right_wheel_link">
+    <visual>
+      <origin xyz="0 0 0" rpy="1.5708 0 0"/>
+      <geometry>
+        <cylinder radius="0.035" length="0.030"/>
+      </geometry>
+      <material name="red_tire">
+        <color rgba="0.85 0.0 0.0 1.0"/>
+      </material>
+    </visual>
+    <visual>
+      <origin xyz="0 0 0.002" rpy="1.5708 0 0"/>
+      <geometry>
+        <cylinder radius="0.020" length="0.040"/>
+      </geometry>
+      <material name="white_rim">
+        <color rgba="1.0 1.0 1.0 1.0"/>
+      </material>
+    </visual>
+    <collision>
+      <origin xyz="0 0 0" rpy="1.5708 0 0"/>
+      <geometry>
+        <cylinder radius="0.035" length="0.039"/>
+      </geometry>
+    </collision>
+  </link>
   <joint name="right_wheel_joint" type="continuous">
     <parent link="base_link"/>
@@ -111,3 +110,90 @@
     <axis xyz="1 0 0"/>
   </joint>
+  <!-- ===================== -->
+  <!-- RIGHT CASTER -->
+  <!-- ===================== -->
+  <link name="right_caster_link">
+    <visual>
+      <geometry>
+        <sphere radius="0.015"/>
+      </geometry>
+      <material name="gray">
+        <color rgba="0.7 0.7 0.7 1.0"/>
+      </material>
+    </visual>
+    <collision>
+      <geometry>
+        <sphere radius="0.015"/>
+      </geometry>
+    </collision>
+  </link>
+  <joint name="right_caster_joint" type="fixed">
+    <parent link="base_link"/>
+    <child link="right_caster_link"/>
+    <origin xyz="0.08 0.0 -0.045"/>
+  </joint>
+  <!-- ===================== -->
+  <!-- LEFT CASTER -->
+  <!-- ===================== -->
+  <link name="left_caster_link">
+    <visual>
+      <geometry>
+        <sphere radius="0.015"/>
+      </geometry>
+      <material name="gray">
+        <color rgba="0.7 0.7 0.7 1.0"/>
+      </material>
+    </visual>
+    <collision>
+      <geometry>
+        <sphere radius="0.015"/>
+      </geometry>
+    </collision>
+  </link>
+  <joint name="left_caster_joint" type="fixed">
+    <parent link="base_link"/>
+    <child link="left_caster_link"/>
+    <origin xyz="-0.08 0.0 -0.045"/>
+  </joint>
+  <!-- ===================== -->
+  <!-- LIDAR MOUNT -->
+  <!-- ===================== -->
+  <link name="lidar_mount_link">
+    <visual>
+      <geometry>
+        <box size="0.06 0.06 0.015"/>
+      </geometry>
+      <material name="dark_gray">
+        <color rgba="0.3 0.3 0.3 1.0"/>
+      </material>
+    </visual>
+    <collision>
+      <geometry>
+        <box size="0.06 0.06 0.015"/>
+      </geometry>
+    </collision>
+  </link>
+  <joint name="lidar_mount_joint" type="fixed">
+    <parent link="base_link"/>
+    <child link="lidar_mount_link"/>
+    <origin xyz="0 0 0.0525"/>
+  </joint>
+  <!-- ===================== -->
+  <!-- LIDAR -->
+  <!-- ===================== -->
+  <link name="lidar_link">
+    <visual>
+      <geometry>
+        <cylinder radius="0.031" length="0.03"/>
+      </geometry>
+      <material name="black">
+        <color rgba="0.05 0.05 0.05 1.0"/>
+      </material>
+    </visual>
+  </link>
+  <joint name="lidar_joint" type="fixed">
+    <parent link="lidar_mount_link"/>
+    <child link="lidar_link"/>
+    <origin xyz="0 0 0.015"/>
+  </joint>
 </robot>

Commit message: seperated main xacro file

File: urdf/hamals_robot.urdf.xacro (robot description, xacro)
@@ -1,199 +1,8 @@
 <?xml version="1.0"?>
 <robot xmlns:xacro="http://www.ros.org/wiki/xacro" name="hamals_robot">
-  <!-- ===================== -->
-  <!-- CHASSIS PROPERTIES -->
-  <!-- ===================== -->
-  <xacro:property name="chassis_length" value="0.22"/>
-  <xacro:property name="chassis_width"  value="0.156"/>
-  <xacro:property name="chassis_height" value="0.09"/>
-  <!-- ===================== -->
-  <!-- BASE FOOTPRINT (Z = 0, zemin referansı) -->
-  <!-- ===================== -->
-  <link name="base_footprint"/>
-  <joint name="base_footprint_joint" type="fixed">
-    <parent link="base_footprint"/>
-    <child link="base_link"/>
-    <origin xyz="0 0 0.045"/>
-  </joint>
-  <!-- ===================== -->
-  <!-- BASE LINK -->
-  <!-- ===================== -->
-  <link name="base_link">
-    <visual>
-      <geometry>
-        <box size="${chassis_length} ${chassis_width} ${chassis_height}"/>
-      </geometry>
-      <material name="navy">
-        <color rgba="0.05 0.1 0.4 1.0"/>
-      </material>
-    </visual>
-    <collision>
-      <geometry>
-        <box size="${chassis_length} ${chassis_width} ${chassis_height}"/>
-      </geometry>
-    </collision>
-    <inertial>
-      <mass value="5.0"/>
-      <inertia ixx="0.02" ixy="0" ixz="0"
-               iyy="0.02" iyz="0"
-               izz="0.02"/>
-    </inertial>
-  </link>
-  <!-- ===================== -->
-  <!-- LEFT WHEEL -->
-  <!-- ===================== -->
-  <link name="left_wheel_link">
-    <visual>
-      <origin xyz="0 0 0" rpy="1.5708 0 0"/>
-      <geometry>
-        <cylinder radius="0.035" length="0.030"/>
-      </geometry>
-      <material name="red_tire">
-        <color rgba="0.85 0.0 0.0 1.0"/>
-      </material>
-    </visual>
-    <visual>
-      <origin xyz="0 0 0.002" rpy="1.5708 0 0"/>
-      <geometry>
-        <cylinder radius="0.020" length="0.040"/>
-      </geometry>
-      <material name="white_rim">
-        <color rgba="1.0 1.0 1.0 1.0"/>
-      </material>
-    </visual>
-    <collision>
-      <origin xyz="0 0 0" rpy="1.5708 0 0"/>
-      <geometry>
-        <cylinder radius="0.035" length="0.039"/>
-      </geometry>
-    </collision>
-  </link>
-  <joint name="left_wheel_joint" type="continuous">
-    <parent link="base_link"/>
-    <child link="left_wheel_link"/>
-    <origin xyz="0 0.095 -0.028"/>
-    <axis xyz="1 0 0"/>
-  </joint>
-  <!-- ===================== -->
-  <!-- RIGHT WHEEL -->
-  <!-- ===================== -->
-  <link name="right_wheel_link">
-    <visual>
-      <origin xyz="0 0 0" rpy="1.5708 0 0"/>
-      <geometry>
-        <cylinder radius="0.035" length="0.030"/>
-      </geometry>
-      <material name="red_tire">
-        <color rgba="0.85 0.0 0.0 1.0"/>
-      </material>
-    </visual>
-    <visual>
-      <origin xyz="0 0 0.002" rpy="1.5708 0 0"/>
-      <geometry>
-        <cylinder radius="0.020" length="0.040"/>
-      </geometry>
-      <material name="white_rim">
-        <color rgba="1.0 1.0 1.0 1.0"/>
-      </material>
-    </visual>
-    <collision>
-      <origin xyz="0 0 0" rpy="1.5708 0 0"/>
-      <geometry>
-        <cylinder radius="0.035" length="0.039"/>
-      </geometry>
-    </collision>
-  </link>
-  <joint name="right_wheel_joint" type="continuous">
-    <parent link="base_link"/>
-    <child link="right_wheel_link"/>
-    <origin xyz="0 -0.095 -0.028"/>
-    <axis xyz="1 0 0"/>
-  </joint>
-  <!-- ===================== -->
-  <!-- RIGHT CASTER -->
-  <!-- ===================== -->
-  <link name="right_caster_link">
-    <visual>
-      <geometry>
-        <sphere radius="0.015"/>
-      </geometry>
-      <material name="gray">
-        <color rgba="0.7 0.7 0.7 1.0"/>
-      </material>
-    </visual>
-    <collision>
-      <geometry>
-        <sphere radius="0.015"/>
-      </geometry>
-    </collision>
-  </link>
-  <joint name="right_caster_joint" type="fixed">
-    <parent link="base_link"/>
-    <child link="right_caster_link"/>
-    <origin xyz="0.08 0.0 -0.045"/>
-  </joint>
-  <!-- ===================== -->
-  <!-- LEFT CASTER -->
-  <!-- ===================== -->
-  <link name="left_caster_link">
-    <visual>
-      <geometry>
-        <sphere radius="0.015"/>
-      </geometry>
-      <material name="gray">
-        <color rgba="0.7 0.7 0.7 1.0"/>
-      </material>
-    </visual>
-    <collision>
-      <geometry>
-        <sphere radius="0.015"/>
-      </geometry>
-    </collision>
-  </link>
-  <joint name="left_caster_joint" type="fixed">
-    <parent link="base_link"/>
-    <child link="left_caster_link"/>
-    <origin xyz="-0.08 0.0 -0.045"/>
-  </joint>
-  <!-- ===================== -->
-  <!-- LIDAR MOUNT -->
-  <!-- ===================== -->
-  <link name="lidar_mount_link">
-    <visual>
-      <geometry>
-        <box size="0.06 0.06 0.015"/>
-      </geometry>
-      <material name="dark_gray">
-        <color rgba="0.3 0.3 0.3 1.0"/>
-      </material>
-    </visual>
-    <collision>
-      <geometry>
-        <box size="0.06 0.06 0.015"/>
-      </geometry>
-    </collision>
-  </link>
-  <joint name="lidar_mount_joint" type="fixed">
-    <parent link="base_link"/>
-    <child link="lidar_mount_link"/>
-    <origin xyz="0 0 0.0525"/>
-  </joint>
-  <!-- ===================== -->
-  <!-- LIDAR -->
-  <!-- ===================== -->
-  <link name="lidar_link">
-    <visual>
-      <geometry>
-        <cylinder radius="0.031" length="0.03"/>
-      </geometry>
-      <material name="black">
-        <color rgba="0.05 0.05 0.05 1.0"/>
-      </material>
-    </visual>
-  </link>
-  <joint name="lidar_joint" type="fixed">
-    <parent link="lidar_mount_link"/>
-    <child link="lidar_link"/>
-    <origin xyz="0 0 0.015"/>
-  </joint>
+  <xacro:include filename="$(find hamals_robot_description)/urdf/materials.xacro"/>
+  <xacro:include filename="$(find hamals_robot_description)/urdf/base.xacro"/>
+  <xacro:include filename="$(find hamals_robot_description)/urdf/wheels.xacro"/>
+  <xacro:include filename="$(find hamals_robot_description)/urdf/casters.xacro"/>
+  <xacro:include filename="$(find hamals_robot_description)/urdf/lidar.xacro"/>
 </robot>

File: urdf/wheels.xacro (robot description, xacro)
@@ -1,47 +1,37 @@
 <?xml version="1.0"?>
 <robot xmlns:xacro="http://www.ros.org/wiki/xacro">
-  <!-- Teker ölçüleri (metre) -->
-  <xacro:property name="wheel_radius" value="0.035"/>   <!-- 3.5 cm -->
-  <xacro:property name="wheel_width"  value="0.039"/>   <!-- 3.9 cm -->
-  <!-- Sol teker macro -->
-  <xacro:macro name="left_wheel">
-    <!-- Sol teker link -->
-    <link name="left_wheel_link">
-      <visual>
-        <origin xyz="0 0 0" rpy="0 0 0"/>
-        <geometry>
-          <cylinder radius="${wheel_radius}" length="${wheel_width}"/>
-        </geometry>
-        <material name="black">
-          <color rgba="0.05 0.05 0.05 1.0"/>
-        </material>
-      </visual>
-      <collision>
-        <origin xyz="0 0 0" rpy="0 0 0"/>
-        <geometry>
-          <cylinder radius="${wheel_radius}" length="${wheel_width}"/>
-        </geometry>
-      </collision>
-      <inertial>
-        <mass value="0.5"/>
-        <origin xyz="0 0 0"/>
-        <inertia
-          ixx="0.001" ixy="0.0" ixz="0.0"
-          iyy="0.001" iyz="0.0"
-          izz="0.001"/>
-      </inertial>
-    </link>
-    <!-- Sol teker joint -->
-    <joint name="left_wheel_joint" type="continuous">
-      <parent link="base_link"/>
-      <child link="left_wheel_link"/>
-      <!-- Konum:
-           X = 0 (şase ortası)
-           Y = +0.09 m (18 cm / 2)
-           Z = 0.035 m (teker yarıçapı) -->
-      <origin xyz="0 0.09 0.035" rpy="0 0 0"/>
-      <!-- Teker X ekseni etrafında döner -->
-      <axis xyz="1 0 0"/>
-    </joint>
-  </xacro:macro>
+  <!-- LEFT WHEEL -->
+  <link name="left_wheel_link">
+    <visual>
+      <origin xyz="0 0 0" rpy="1.5708 0 0"/>
+      <geometry>
+        <cylinder radius="0.035" length="0.030"/>
+      </geometry>
+      <!-- SADECE REFERANS -->
+      <material name="wheel_red"/>
+    </visual>
+  </link>
+  <joint name="left_wheel_joint" type="continuous">
+    <parent link="base_link"/>
+    <child link="left_wheel_link"/>
+    <origin xyz="0 0.095 -0.028"/>
+    <axis xyz="1 0 0"/>
+  </joint>
+  <!-- RIGHT WHEEL -->
+  <link name="right_wheel_link">
+    <visual>
+      <origin xyz="0 0 0" rpy="1.5708 0 0"/>
+      <geometry>
+        <cylinder radius="0.035" length="0.030"/>
+      </geometry>
+      <!-- SADECE REFERANS -->
+      <material name="wheel_red"/>
+    </visual>
+  </link>
+  <joint name="right_wheel_joint" type="continuous">
+    <parent link="base_link"/>
+    <child link="right_wheel_link"/>
+    <origin xyz="0 -0.095 -0.028"/>
+    <axis xyz="1 0 0"/>
+  </joint>
 </robot>
