Commit message: Finalize robot description: geometry, wheels, casters, lidar mounting

File: urdf/base.xacro (robot description, xacro)
@@ -1,22 +1,36 @@
 <?xml version="1.0"?>
 <robot xmlns:xacro="http://www.ros.org/wiki/xacro">
-  <xacro:property name="chassis_length" value="0.22"/>
-  <xacro:property name="chassis_width"  value="0.156"/>
-  <xacro:property name="chassis_height" value="0.09"/>
+  <!-- ================================================= -->
+  <!-- Load robot dimensions from YAML (single source) -->
+  <!-- ================================================= -->
+  <xacro:property name="dims"
+    value="${xacro.load_yaml('$(find hamals_robot_description)/config/robot_dimensions.yaml')}" />
+  <!-- Chassis dimensions -->
+  <xacro:property name="chassis_length" value="${dims['robot']['length']}"/>
+  <xacro:property name="chassis_width"  value="${dims['robot']['width']}"/>
+  <xacro:property name="chassis_height" value="${dims['robot']['height']}"/>
+  <!-- Base frame height -->
+  <xacro:property name="base_link_z" value="${dims['base_frames']['base_link_z']}"/>
+  <!-- ================================================= -->
+  <!-- Base Footprint (2D reference frame)               -->
+  <!-- ================================================= -->
   <link name="base_footprint"/>
+  <!-- ================================================= -->
+  <!-- Base Link                                        -->
+  <!-- ================================================= -->
   <joint name="base_footprint_joint" type="fixed">
     <parent link="base_footprint"/>
     <child link="base_link"/>
-    <origin xyz="0 0 0.045"/>
+    <origin xyz="0 0 ${base_link_z}"/>
   </joint>
   <link name="base_link">
+    <!-- Visual geometry -->
     <visual>
       <geometry>
         <box size="${chassis_length} ${chassis_width} ${chassis_height}"/>
       </geometry>
-      <material name="navy">
-        <color rgba="0.05 0.1 0.4 1.0"/>
-      </material>
+      <material name="navy"/>
     </visual>
+    <!-- Collision geometry (same as chassis for now) -->
     <collision>
       <geometry>
@@ -24,9 +38,11 @@
       </geometry>
     </collision>
+    <!-- Inertial (simple, acceptable for now) -->
     <inertial>
-      <mass value="5.0"/>
-      <inertia ixx="0.02" ixy="0" ixz="0"
-               iyy="0.02" iyz="0"
-               izz="0.02"/>
+      <mass value="${dims['robot']['mass']}"/>
+      <inertia
+        ixx="0.02" ixy="0.0" ixz="0.0"
+        iyy="0.02" iyz="0.0"
+        izz="0.02"/>
     </inertial>
   </link>

File: urdf/casters.xacro (robot description, xacro)
@@ -1,47 +1,51 @@
 <?xml version="1.0"?>
 <robot xmlns:xacro="http://www.ros.org/wiki/xacro">
-  <!-- ===================== -->
-  <!-- RIGHT CASTER -->
-  <!-- ===================== -->
-  <link name="right_caster_link">
+  <xacro:property name="dims"
+    value="${xacro.load_yaml('$(find hamals_robot_description)/config/robot_dimensions.yaml')}" />
+  <!-- Drive wheel geometry (AUTHORITATIVE ground reference) -->
+  <xacro:property name="wheel_radius"
+    value="${dims['wheels']['radius']}"/>
+  <xacro:property name="wheel_center_z"
+    value="${dims['wheels']['z_offset'] * -1.0}"/>
+  <!-- Caster geometry -->
+  <xacro:property name="caster_radius"
+    value="${dims['casters']['radius']}"/>
+  <xacro:property name="front_x"
+    value="${dims['casters']['front_x']}"/>
+  <xacro:property name="rear_x"
+    value="${dims['casters']['rear_x']}"/>
+  <!-- Ground plane from wheel -->
+  <xacro:property name="ground_z"
+    value="${wheel_center_z - wheel_radius}"/>
+  <!-- Caster center exactly touching ground -->
+  <xacro:property name="caster_z"
+    value="${ground_z + caster_radius}"/>
+  <!-- FRONT CASTER -->
+  <link name="front_caster_link">
     <visual>
       <geometry>
-        <sphere radius="0.015"/>
+        <sphere radius="${caster_radius}"/>
       </geometry>
-      <!-- MATERIAL REFERANSI -->
       <material name="caster_gray"/>
     </visual>
-    <collision>
-      <geometry>
-        <sphere radius="0.015"/>
-      </geometry>
-    </collision>
   </link>
-  <joint name="right_caster_joint" type="fixed">
+  <joint name="front_caster_joint" type="fixed">
     <parent link="base_link"/>
-    <child link="right_caster_link"/>
-    <origin xyz="0.08 0.0 -0.045"/>
+    <child link="front_caster_link"/>
+    <origin xyz="${front_x} 0 ${caster_z}"/>
   </joint>
-  <!-- ===================== -->
-  <!-- LEFT CASTER -->
-  <!-- ===================== -->
-  <link name="left_caster_link">
+  <!-- REAR CASTER -->
+  <link name="rear_caster_link">
     <visual>
       <geometry>
-        <sphere radius="0.015"/>
+        <sphere radius="${caster_radius}"/>
       </geometry>
-      <!-- MATERIAL REFERANSI -->
       <material name="caster_gray"/>
     </visual>
-    <collision>
-      <geometry>
-        <sphere radius="0.015"/>
-      </geometry>
-    </collision>
   </link>
-  <joint name="left_caster_joint" type="fixed">
+  <joint name="rear_caster_joint" type="fixed">
     <parent link="base_link"/>
-    <child link="left_caster_link"/>
-    <origin xyz="-0.08 0.0 -0.045"/>
+    <child link="rear_caster_link"/>
+    <origin xyz="${rear_x} 0 ${caster_z}"/>
   </joint>
 </robot>

File: urdf/hamals_robot.urdf.xacro (robot description, xacro)
@@ -1,5 +1,16 @@
 <?xml version="1.0"?>
 <robot xmlns:xacro="http://www.ros.org/wiki/xacro" name="hamals_robot">
+  <!-- ================================================= -->
+  <!-- Load robot dimensions ONCE (global scope)        -->
+  <!-- ================================================= -->
+  <xacro:property name="dims"
+    value="${xacro.load_yaml('$(find hamals_robot_description)/config/robot_dimensions.yaml')}" />
+  <!-- ================================================= -->
+  <!-- Materials                                        -->
+  <!-- ================================================= -->
   <xacro:include filename="$(find hamals_robot_description)/urdf/materials.xacro"/>
+  <!-- ================================================= -->
+  <!-- Robot Structure                                  -->
+  <!-- ================================================= -->
   <xacro:include filename="$(find hamals_robot_description)/urdf/base.xacro"/>
   <xacro:include filename="$(find hamals_robot_description)/urdf/wheels.xacro"/>

File: urdf/lidar.xacro (robot description, xacro)
@@ -1,42 +1,69 @@
 <?xml version="1.0"?>
 <robot xmlns:xacro="http://www.ros.org/wiki/xacro">
-  <!-- ===================== -->
-  <!-- LIDAR MOUNT -->
-  <!-- ===================== -->
+  <!-- ================================================= -->
+  <!-- Load robot dimensions from YAML                  -->
+  <!-- ================================================= -->
+  <xacro:property name="dims"
+    value="${xacro.load_yaml('$(find hamals_robot_description)/config/robot_dimensions.yaml')}" />
+  <!-- Base frame height -->
+  <xacro:property name="base_link_z"
+    value="${dims['base_frames']['base_link_z']}"/>
+  <!-- Lidar parameters -->
+  <xacro:property name="lidar_height"
+    value="${dims['lidar']['height']}"/>
+  <xacro:property name="lidar_offset_x"
+    value="${dims['lidar']['offset']['x']}"/>
+  <xacro:property name="lidar_offset_y"
+    value="${dims['lidar']['offset']['y']}"/>
+  <!-- Lidar geometry -->
+  <xacro:property name="lidar_body_length" value="0.03"/>
+  <xacro:property name="lidar_body_radius" value="0.031"/>
+  <!-- Mount geometry -->
+  <xacro:property name="mount_thickness" value="0.015"/>
+  <xacro:property name="mount_gap"
+    value="${dims['lidar']['mount']['gap']}"/>
+  <!-- ================================================= -->
+  <!-- LIDAR LINK (REFERENCE SENSOR)                     -->
+  <!-- ================================================= -->
+  <link name="lidar_link">
+    <visual>
+      <geometry>
+        <cylinder radius="${lidar_body_radius}"
+                  length="${lidar_body_length}"/>
+      </geometry>
+      <material name="lidar_black"/>
+    </visual>
+  </link>
+  <!-- Lidar center placed exactly at lidar_height -->
+  <xacro:property name="lidar_z"
+    value="${lidar_height - base_link_z}"/>
+  <joint name="lidar_joint" type="fixed">
+    <parent link="base_link"/>
+    <child link="lidar_link"/>
+    <origin
+      xyz="${lidar_offset_x} ${lidar_offset_y} ${lidar_z}"/>
+  </joint>
+  <!-- ================================================= -->
+  <!-- LIDAR MOUNT (JUST BELOW LIDAR)                    -->
+  <!-- ================================================= -->
   <link name="lidar_mount_link">
     <visual>
       <geometry>
-        <box size="0.06 0.06 0.015"/>
+        <box size="0.06 0.06 ${mount_thickness}"/>
       </geometry>
-      <!-- MATERIAL REFERANSI -->
       <material name="lidar_mount_gray"/>
     </visual>
     <collision>
       <geometry>
-        <box size="0.06 0.06 0.015"/>
+        <box size="0.06 0.06 ${mount_thickness}"/>
       </geometry>
     </collision>
   </link>
+  <xacro:property name="mount_offset_z"
+    value="${-(lidar_body_length/2.0 + mount_thickness/2.0 - mount_gap)}"/>
   <joint name="lidar_mount_joint" type="fixed">
-    <parent link="base_link"/>
+    <parent link="lidar_link"/>
     <child link="lidar_mount_link"/>
-    <origin xyz="0 0 0.0525"/>
-  </joint>
-  <!-- ===================== -->
-  <!-- LIDAR -->
-  <!-- ===================== -->
-  <link name="lidar_link">
-    <visual>
-      <geometry>
-        <cylinder radius="0.031" length="0.03"/>
-      </geometry>
-      <!-- MATERIAL REFERANSI -->
-      <material name="lidar_black"/>
-    </visual>
-  </link>
-  <joint name="lidar_joint" type="fixed">
-    <parent link="lidar_mount_link"/>
-    <child link="lidar_link"/>
-    <origin xyz="0 0 0.015"/>
+    <origin xyz="0 0 ${mount_offset_z}"/>
   </joint>
 </robot>

File: urdf/wheels.xacro (robot description, xacro)
@@ -1,12 +1,23 @@
 <?xml version="1.0"?>
 <robot xmlns:xacro="http://www.ros.org/wiki/xacro">
-  <!-- LEFT WHEEL -->
+  <!-- ================================================= -->
+  <!-- Load robot dimensions from YAML                  -->
+  <!-- ================================================= -->
+  <xacro:property name="dims"
+    value="${xacro.load_yaml('$(find hamals_robot_description)/config/robot_dimensions.yaml')}" />
+  <!-- Wheel parameters -->
+  <xacro:property name="wheel_radius"    value="${dims['wheels']['radius']}"/>
+  <xacro:property name="wheel_thickness" value="${dims['wheels']['thickness']}"/>
+  <xacro:property name="wheel_sep"       value="${dims['wheels']['separation']}"/>
+  <!-- ================================================= -->
+  <!-- LEFT WHEEL                                       -->
+  <!-- ================================================= -->
   <link name="left_wheel_link">
     <visual>
+      <!-- Rotate cylinder so axis aligns with wheel axle -->
       <origin xyz="0 0 0" rpy="1.5708 0 0"/>
       <geometry>
-        <cylinder radius="0.035" length="0.030"/>
+        <cylinder radius="${wheel_radius}" length="${wheel_thickness}"/>
       </geometry>
-      <!-- SADECE REFERANS -->
       <material name="wheel_red"/>
     </visual>
@@ -15,15 +26,17 @@
     <parent link="base_link"/>
     <child link="left_wheel_link"/>
-    <origin xyz="0 0.095 -0.028"/>
+    <!-- y = +wheel_sep/2 , z = -wheel_radius -->
+    <origin xyz="0 ${wheel_sep / 2.0} ${-wheel_radius}"/>
     <axis xyz="1 0 0"/>
   </joint>
-  <!-- RIGHT WHEEL -->
+  <!-- ================================================= -->
+  <!-- RIGHT WHEEL                                      -->
+  <!-- ================================================= -->
   <link name="right_wheel_link">
     <visual>
       <origin xyz="0 0 0" rpy="1.5708 0 0"/>
       <geometry>
-        <cylinder radius="0.035" length="0.030"/>
+        <cylinder radius="${wheel_radius}" length="${wheel_thickness}"/>
       </geometry>
-      <!-- SADECE REFERANS -->
       <material name="wheel_red"/>
     </visual>
@@ -32,5 +45,6 @@
     <parent link="base_link"/>
     <child link="right_wheel_link"/>
-    <origin xyz="0 -0.095 -0.028"/>
+    <!-- y = -wheel_sep/2 , z = -wheel_radius -->
+    <origin xyz="0 ${-wheel_sep / 2.0} ${-wheel_radius}"/>
     <axis xyz="1 0 0"/>
   </joint>

Commit message: Refactor robot description launch and xacro structure

File: urdf/base.xacro (robot description, xacro)
@@ -1,49 +1,41 @@
 <?xml version="1.0"?>
 <robot xmlns:xacro="http://www.ros.org/wiki/xacro">
-  <!-- ================================================= -->
-  <!-- Load robot dimensions from YAML (single source) -->
-  <!-- ================================================= -->
-  <xacro:property name="dims"
-    value="${xacro.load_yaml('$(find hamals_robot_description)/config/robot_dimensions.yaml')}" />
-  <!-- Chassis dimensions -->
-  <xacro:property name="chassis_length" value="${dims['robot']['length']}"/>
-  <xacro:property name="chassis_width"  value="${dims['robot']['width']}"/>
-  <xacro:property name="chassis_height" value="${dims['robot']['height']}"/>
-  <!-- Base frame height -->
-  <xacro:property name="base_link_z" value="${dims['base_frames']['base_link_z']}"/>
-  <!-- ================================================= -->
-  <!-- Base Footprint (2D reference frame)               -->
-  <!-- ================================================= -->
-  <link name="base_footprint"/>
-  <!-- ================================================= -->
-  <!-- Base Link                                        -->
-  <!-- ================================================= -->
-  <joint name="base_footprint_joint" type="fixed">
-    <parent link="base_footprint"/>
-    <child link="base_link"/>
-    <origin xyz="0 0 ${base_link_z}"/>
-  </joint>
-  <link name="base_link">
-    <!-- Visual geometry -->
-    <visual>
-      <geometry>
-        <box size="${chassis_length} ${chassis_width} ${chassis_height}"/>
-      </geometry>
-      <material name="navy"/>
-    </visual>
-    <!-- Collision geometry (same as chassis for now) -->
-    <collision>
-      <geometry>
-        <box size="${chassis_length} ${chassis_width} ${chassis_height}"/>
-      </geometry>
-    </collision>
-    <!-- Inertial (simple, acceptable for now) -->
-    <inertial>
-      <mass value="${dims['robot']['mass']}"/>
-      <inertia
-        ixx="0.02" ixy="0.0" ixz="0.0"
-        iyy="0.02" iyz="0.0"
-        izz="0.02"/>
-    </inertial>
-  </link>
+  <xacro:macro name="hamals_base" params="config">
+    <!-- Zemindeki ana referans frame -->
+    <link name="${config['robot']['frames']['base_footprint']}"/>
+    <!-- Gövde merkezi -->
+    <joint name="base_footprint_to_base_link" type="fixed">
+      <parent link="${config['robot']['frames']['base_footprint']}"/>
+      <child link="${config['robot']['frames']['base_link']}"/>
+      <origin
+        xyz="${config['base']['origin']['xyz'][0]} ${config['base']['origin']['xyz'][1]} ${config['base']['origin']['xyz'][2]}"
+        rpy="${config['base']['origin']['rpy'][0]} ${config['base']['origin']['rpy'][1]} ${config['base']['origin']['rpy'][2]}"/>
+    </joint>
+    <link name="${config['robot']['frames']['base_link']}">
+      <visual>
+        <origin xyz="0 0 0" rpy="0 0 0"/>
+        <geometry>
+          <box size="${config['base']['length']} ${config['base']['width']} ${config['base']['height']}"/>
+        </geometry>
+        <material name="${config['materials']['base']['name']}"/>
+      </visual>
+      <collision>
+        <origin xyz="0 0 0" rpy="0 0 0"/>
+        <geometry>
+          <box size="${config['base']['collision']['length']} ${config['base']['collision']['width']} ${config['base']['collision']['height']}"/>
+        </geometry>
+      </collision>
+      <inertial>
+        <origin xyz="0 0 0" rpy="0 0 0"/>
+        <mass value="${config['inertial']['base']['mass']}"/>
+        <inertia
+          ixx="${config['inertial']['base']['ixx']}"
+          ixy="${config['inertial']['base']['ixy']}"
+          ixz="${config['inertial']['base']['ixz']}"
+          iyy="${config['inertial']['base']['iyy']}"
+          iyz="${config['inertial']['base']['iyz']}"
+          izz="${config['inertial']['base']['izz']}"/>
+      </inertial>
+    </link>
+  </xacro:macro>
 </robot>

File: urdf/hamals_robot.urdf.xacro (robot description, xacro)
@@ -1,19 +1,8 @@
 <?xml version="1.0"?>
-<robot xmlns:xacro="http://www.ros.org/wiki/xacro" name="hamals_robot">
-  <!-- ================================================= -->
-  <!-- Load robot dimensions ONCE (global scope)        -->
-  <!-- ================================================= -->
-  <xacro:property name="dims"
-    value="${xacro.load_yaml('$(find hamals_robot_description)/config/robot_dimensions.yaml')}" />
-  <!-- ================================================= -->
-  <!-- Materials                                        -->
-  <!-- ================================================= -->
+<robot name="hamals_robot" xmlns:xacro="http://www.ros.org/wiki/xacro">
+  <xacro:property name="config" value="${xacro.load_yaml('$(find hamals_robot_description)/config/robot_dimensions.yaml')}"/>
   <xacro:include filename="$(find hamals_robot_description)/urdf/materials.xacro"/>
-  <!-- ================================================= -->
-  <!-- Robot Structure                                  -->
-  <!-- ================================================= -->
   <xacro:include filename="$(find hamals_robot_description)/urdf/base.xacro"/>
-  <xacro:include filename="$(find hamals_robot_description)/urdf/wheels.xacro"/>
-  <xacro:include filename="$(find hamals_robot_description)/urdf/casters.xacro"/>
-  <xacro:include filename="$(find hamals_robot_description)/urdf/lidar.xacro"/>
+  <xacro:hamals_materials config="${config}"/>
+  <xacro:hamals_base config="${config}"/>
 </robot>

File: urdf/materials.xacro (robot description, xacro)
@@ -1,33 +1,29 @@
 <?xml version="1.0"?>
 <robot xmlns:xacro="http://www.ros.org/wiki/xacro">
-  <!-- ===================== -->
-  <!-- CHASSIS -->
-  <!-- ===================== -->
-  <material name="navy">
-    <color rgba="0.05 0.1 0.4 1.0"/>
-  </material>
-  <!-- ===================== -->
-  <!-- WHEELS -->
-  <!-- ===================== -->
-  <material name="wheel_red">
-    <color rgba="0.85 0.0 0.0 1.0"/>
-  </material>
-  <material name="wheel_rim_white">
-    <color rgba="1.0 1.0 1.0 1.0"/>
-  </material>
-  <!-- ===================== -->
-  <!-- CASTERS -->
-  <!-- ===================== -->
-  <material name="caster_gray">
-    <color rgba="0.7 0.7 0.7 1.0"/>
-  </material>
-  <!-- ===================== -->
-  <!-- LIDAR -->
-  <!-- ===================== -->
-  <material name="lidar_black">
-    <color rgba="0.05 0.05 0.05 1.0"/>
-  </material>
-  <material name="lidar_mount_gray">
-    <color rgba="0.3 0.3 0.3 1.0"/>
-  </material>
+  <xacro:macro name="hamals_materials" params="config">
+    <material name="${config['materials']['base']['name']}">
+      <color rgba="${' '.join([str(x) for x in config['materials']['base']['color']])}"/>
+    </material>
+    <material name="${config['materials']['wheels']['name']}">
+      <color rgba="${' '.join([str(x) for x in config['materials']['wheels']['color']])}"/>
+    </material>
+    <material name="${config['materials']['caster']['name']}">
+      <color rgba="${' '.join([str(x) for x in config['materials']['caster']['color']])}"/>
+    </material>
+    <material name="${config['materials']['lidar_mount']['name']}">
+      <color rgba="${' '.join([str(x) for x in config['materials']['lidar_mount']['color']])}"/>
+    </material>
+    <material name="${config['materials']['lidar']['name']}">
+      <color rgba="${' '.join([str(x) for x in config['materials']['lidar']['color']])}"/>
+    </material>
+    <material name="${config['materials']['forklift_mast']['name']}">
+      <color rgba="${' '.join([str(x) for x in config['materials']['forklift_mast']['color']])}"/>
+    </material>
+    <material name="${config['materials']['fork_carriage']['name']}">
+      <color rgba="${' '.join([str(x) for x in config['materials']['fork_carriage']['color']])}"/>
+    </material>
+    <material name="${config['materials']['forks']['name']}">
+      <color rgba="${' '.join([str(x) for x in config['materials']['forks']['color']])}"/>
+    </material>
+  </xacro:macro>
 </robot>
