Commit message: Refine forklift AGV geometry and joint publishing

File: urdf/wheels.xacro (robot description, xacro)
@@ -2,21 +2,21 @@
 <robot xmlns:xacro="http://www.ros.org/wiki/xacro">
   <xacro:macro name="hamals_wheels" params="config">
-    <!-- Arka sol ana sürüş tekeri -->
-    <joint name="${config['wheels']['rear_left']['joint']['name']}" type="${config['wheels']['rear_left']['joint']['type']}">
-      <parent link="${config['wheels']['rear_left']['joint']['parent']}"/>
-      <child link="${config['wheels']['rear_left']['joint']['child']}"/>
+    <!-- Sol ana sürüş tekeri -->
+    <joint name="${config['wheels']['left_drive']['joint']['name']}" type="${config['wheels']['left_drive']['joint']['type']}">
+      <parent link="${config['wheels']['left_drive']['joint']['parent']}"/>
+      <child link="${config['wheels']['left_drive']['joint']['child']}"/>
       <origin
-        xyz="${config['wheels']['rear_left']['origin']['xyz'][0]} ${config['wheels']['rear_left']['origin']['xyz'][1]} ${config['wheels']['rear_left']['origin']['xyz'][2]}"
-        rpy="${config['wheels']['rear_left']['origin']['rpy'][0]} ${config['wheels']['rear_left']['origin']['rpy'][1]} ${config['wheels']['rear_left']['origin']['rpy'][2]}"/>
+        xyz="${config['wheels']['left_drive']['origin']['xyz'][0]} ${config['wheels']['left_drive']['origin']['xyz'][1]} ${config['wheels']['left_drive']['origin']['xyz'][2]}"
+        rpy="${config['wheels']['left_drive']['origin']['rpy'][0]} ${config['wheels']['left_drive']['origin']['rpy'][1]} ${config['wheels']['left_drive']['origin']['rpy'][2]}"/>
       <axis
-        xyz="${config['wheels']['rear_left']['joint']['axis'][0]} ${config['wheels']['rear_left']['joint']['axis'][1]} ${config['wheels']['rear_left']['joint']['axis'][2]}"/>
+        xyz="${config['wheels']['left_drive']['joint']['axis'][0]} ${config['wheels']['left_drive']['joint']['axis'][1]} ${config['wheels']['left_drive']['joint']['axis'][2]}"/>
     </joint>
-    <link name="${config['robot']['frames']['rear_left_wheel_link']}">
+    <link name="${config['robot']['frames']['left_drive_wheel_link']}">
       <visual>
         <origin xyz="0 0 0" rpy="0 0 0"/>
         <geometry>
           <cylinder
-            radius="${config['wheels']['rear_left']['radius']}"
-            length="${config['wheels']['rear_left']['width']}"/>
+            radius="${config['wheels']['left_drive']['radius']}"
+            length="${config['wheels']['left_drive']['width']}"/>
         </geometry>
         <material name="${config['materials']['wheels']['name']}"/>
@@ -26,6 +26,6 @@
         <geometry>
           <cylinder
-            radius="${config['wheels']['rear_left']['radius']}"
-            length="${config['wheels']['rear_left']['width']}"/>
+            radius="${config['wheels']['left_drive']['radius']}"
+            length="${config['wheels']['left_drive']['width']}"/>
         </geometry>
       </collision>
@@ -42,21 +42,21 @@
       </inertial>
     </link>
-    <!-- Arka sağ ana sürüş tekeri -->
-    <joint name="${config['wheels']['rear_right']['joint']['name']}" type="${config['wheels']['rear_right']['joint']['type']}">
-      <parent link="${config['wheels']['rear_right']['joint']['parent']}"/>
-      <child link="${config['wheels']['rear_right']['joint']['child']}"/>
+    <!-- Sağ ana sürüş tekeri -->
+    <joint name="${config['wheels']['right_drive']['joint']['name']}" type="${config['wheels']['right_drive']['joint']['type']}">
+      <parent link="${config['wheels']['right_drive']['joint']['parent']}"/>
+      <child link="${config['wheels']['right_drive']['joint']['child']}"/>
       <origin
-        xyz="${config['wheels']['rear_right']['origin']['xyz'][0]} ${config['wheels']['rear_right']['origin']['xyz'][1]} ${config['wheels']['rear_right']['origin']['xyz'][2]}"
-        rpy="${config['wheels']['rear_right']['origin']['rpy'][0]} ${config['wheels']['rear_right']['origin']['rpy'][1]} ${config['wheels']['rear_right']['origin']['rpy'][2]}"/>
+        xyz="${config['wheels']['right_drive']['origin']['xyz'][0]} ${config['wheels']['right_drive']['origin']['xyz'][1]} ${config['wheels']['right_drive']['origin']['xyz'][2]}"
+        rpy="${config['wheels']['right_drive']['origin']['rpy'][0]} ${config['wheels']['right_drive']['origin']['rpy'][1]} ${config['wheels']['right_drive']['origin']['rpy'][2]}"/>
       <axis
-        xyz="${config['wheels']['rear_right']['joint']['axis'][0]} ${config['wheels']['rear_right']['joint']['axis'][1]} ${config['wheels']['rear_right']['joint']['axis'][2]}"/>
+        xyz="${config['wheels']['right_drive']['joint']['axis'][0]} ${config['wheels']['right_drive']['joint']['axis'][1]} ${config['wheels']['right_drive']['joint']['axis'][2]}"/>
     </joint>
-    <link name="${config['robot']['frames']['rear_right_wheel_link']}">
+    <link name="${config['robot']['frames']['right_drive_wheel_link']}">
       <visual>
         <origin xyz="0 0 0" rpy="0 0 0"/>
         <geometry>
           <cylinder
-            radius="${config['wheels']['rear_right']['radius']}"
-            length="${config['wheels']['rear_right']['width']}"/>
+            radius="${config['wheels']['right_drive']['radius']}"
+            length="${config['wheels']['right_drive']['width']}"/>
         </geometry>
         <material name="${config['materials']['wheels']['name']}"/>
@@ -66,6 +66,6 @@
         <geometry>
           <cylinder
-            radius="${config['wheels']['rear_right']['radius']}"
-            length="${config['wheels']['rear_right']['width']}"/>
+            radius="${config['wheels']['right_drive']['radius']}"
+            length="${config['wheels']['right_drive']['width']}"/>
         </geometry>
       </collision>
